Commit message: dfdcvc

File: src/tf_publisher_radar/urdf/multi_radars_each_pub.urdf (robot description, URDF)
Before this commit: robot morning_car, 7 links, 6 joints
Links:
- added link RADARS; visual box size=0.05 0.05 0.05
Joints:
- added joint base_au_radar_unified: type fixed, parent base_link, child RADARS, origin xyz=0 0 0 rpy=0 0 0

File: src/tf_publisher_radar/urdf/multi_radars_each_pub_jig.urdf (robot description, URDF)
Before this commit: robot morning_car, 7 links, 6 joints
Links:
- added link RADARS; visual box size=0.05 0.05 0.05
Joints:
- added joint base_au_radar_unified: type fixed, parent base_link, child RADARS, origin xyz=0 0 0 rpy=0 0 0
